Commit message: failed attempt to climb stairs

File: body.urdf (robot description, URDF)
Before this commit: robot robot, 9 links, 8 joints
Links:
- removed link BackLeg
- removed link BackLowerLeg
- removed link FrontLeg
- removed link FrontLowerLeg
- removed link LeftLeg
- removed link LeftLowerLeg
- removed link RightLeg
- removed link RightLowerLeg
- added link LeftLeg1, mass 1; collision box size=1 0.2 0.2; visual box size=1 0.2 0.2
- added link LeftLowerLeg1, mass 1; collision box size=0.2 0.2 0.5; visual box size=0.2 0.2 0.5
- link Torso: geometry collision box size=1 1 0.5; visual box size=1 1 0.5
Joints:
- removed joint BackLeg_BackLowerLeg
- removed joint FrontLeg_FrontLowerLeg
- removed joint LeftLeg_LeftLowerLeg
- removed joint RightLeg_RightLowerLeg
- removed joint Torso_BackLeg
- removed joint Torso_FrontLeg
- removed joint Torso_LeftLeg
- removed joint Torso_RightLeg
- added joint LeftLeg1_LeftLowerLeg1: type revolute, parent LeftLeg1, child LeftLowerLeg1, origin xyz=1 0 0 rpy=0 0 0, axis 0 1 0, limit lower=-3.14159 upper=3.14159 effort=0.0 velocity=0.0
- added joint Torso_LeftLeg1: type revolute, parent Torso, child LeftLeg1, origin xyz=0.5 0 0.5 rpy=0 0 0, axis 0 1 0, limit lower=-3.14159 upper=3.14159 effort=0.0 velocity=0.0

Commit message: finished random vs evolved

File: body.urdf (robot description, URDF)
Before this commit: robot robot, 9 links, 8 joints
Links:
- removed link BackLeg
- removed link BackLowerLeg
- removed link FrontLeg
- removed link FrontLowerLeg
- removed link LeftLeg
- removed link LeftLowerLeg
- removed link RightLeg
- removed link RightLowerLeg
- added link LeftLeg1, mass 1; collision box size=0.5 0.2 0.2; visual box size=0.5 0.2 0.2
- added link LeftLeg2, mass 1; collision box size=0.5 0.2 0.2; visual box size=0.5 0.2 0.2
- added link LeftLowerLeg1, mass 1; collision box size=0.2 0.2 0.5; visual box size=0.2 0.2 0.5
- added link LeftLowerLeg2, mass 1; collision box size=0.2 0.2 0.5; visual box size=0.2 0.2 0.5
- added link RightLeg1, mass 1; collision box size=0.5 0.2 0.2; visual box size=0.5 0.2 0.2
- added link RightLeg2, mass 1; collision box size=0.5 0.2 0.2; visual box size=0.5 0.2 0.2
- added link RightLowerLeg1, mass 1; collision box size=0.2 0.2 0.5; visual box size=0.2 0.2 0.5
- added link RightLowerLeg2, mass 1; collision box size=0.2 0.2 0.5; visual box size=0.2 0.2 0.5
- added link SideArm1, mass 1; collision box size=0.2 0.2 0.2; visual box size=0.2 0.2 0.2
- added link SideArm2, mass 1; collision box size=0.2 0.2 0.2; visual box size=0.2 0.2 0.2
- added link SideLowerArm1, mass 1; collision box size=0.2 0.2 0.8; visual box size=0.2 0.2 0.8
- added link SideLowerArm2, mass 1; collision box size=0.2 0.2 0.8; visual box size=0.2 0.2 0.8
- link Torso: geometry collision box size=1 1 0.5; visual box size=1 1 0.5
Joints:
- removed joint BackLeg_BackLowerLeg
- removed joint FrontLeg_FrontLowerLeg
- removed joint LeftLeg_LeftLowerLeg
- removed joint RightLeg_RightLowerLeg
- removed joint Torso_BackLeg
- removed joint Torso_FrontLeg
- removed joint Torso_LeftLeg
- removed joint Torso_RightLeg
- added joint LeftLeg1_LeftLowerLeg1: type revolute, parent LeftLeg1, child LeftLowerLeg1, origin xyz=0.5 0 0 rpy=0 0 0, axis 0 1 0, limit lower=-3.14159 upper=3.14159 effort=0.0 velocity=0.0
- added joint LeftLeg2_LeftLowerLeg2: type revolute, parent LeftLeg2, child LeftLowerLeg2, origin xyz=0.5 0 0 rpy=0 0 0, axis 0 1 0, limit lower=-3.14159 upper=3.14159 effort=0.0 velocity=0.0
- added joint RightLeg1_RightLowerLeg1: type revolute, parent RightLeg1, child RightLowerLeg1, origin xyz=-0.5 0 0 rpy=0 0 0, axis 0 1 0, limit lower=-3.14159 upper=3.14159 effort=0.0 velocity=0.0
- added joint RightLeg2_RightLowerLeg2: type revolute, parent RightLeg2, child RightLowerLeg2, origin xyz=-0.5 0 0 rpy=0 0 0, axis 0 1 0, limit lower=-3.14159 upper=3.14159 effort=0.0 velocity=0.0
- added joint SideArm1_SideLowerArm1: type revolute, parent SideArm1, child SideLowerArm1, origin xyz=0 -0.2 0 rpy=0 0 0, axis 1 0 0, limit lower=-3.14159 upper=3.14159 effort=0.0 velocity=0.0
- added joint SideArm2_SideLowerArm2: type revolute, parent SideArm2, child SideLowerArm2, origin xyz=0 0.2 0 rpy=0 0 0, axis 1 0 0, limit lower=-3.14159 upper=3.14159 effort=0.0 velocity=0.0
- added joint Torso_LeftLeg1: type revolute, parent Torso, child LeftLeg1, origin xyz=0.5 0.25 2.6 rpy=0 0 0, axis 0 1 0, limit lower=-3.14159 upper=3.14159 effort=0.0 velocity=0.0
- added joint Torso_LeftLeg2: type revolute, parent Torso, child LeftLeg2, origin xyz=0.5 -0.25 2.6 rpy=0 0 0, axis 0 1 0, limit lower=-3.14159 upper=3.14159 effort=0.0 velocity=0.0
- added joint Torso_RightLeg1: type revolute, parent Torso, child RightLeg1, origin xyz=-0.5 0.25 2.6 rpy=0 0 0, axis 0 1 0, limit lower=-3.14159 upper=3.14159 effort=0.0 velocity=0.0
- added joint Torso_RightLeg2: type revolute, parent Torso, child RightLeg2, origin xyz=-0.5 -0.25 2.6 rpy=0 0 0, axis 0 1 0, limit lower=-3.14159 upper=3.14159 effort=0.0 velocity=0.0
- added joint Torso_SideArm1: type revolute, parent Torso, child SideArm1, origin xyz=0 -0.5 2.6 rpy=0 0 0, axis 1 0 0, limit lower=-3.14159 upper=3.14159 effort=0.0 velocity=0.0
- added joint Torso_SideArm2: type revolute, parent Torso, child SideArm2, origin xyz=0 0.5 2.6 rpy=0 0 0, axis 1 0 0, limit lower=-3.14159 upper=3.14159 effort=0.0 velocity=0.0

Commit message: finished random snake

File: body.urdf (robot description, URDF)
Before this commit: robot robot, 13 links, 12 joints
Links:
- removed link LeftLeg1
- removed link LeftLeg2
- removed link LeftLowerLeg1
- removed link LeftLowerLeg2
- removed link RightLeg1
- removed link RightLeg2
- removed link RightLowerLeg1
- removed link RightLowerLeg2
- removed link SideArm1
- removed link SideArm2
- removed link SideLowerArm1
- removed link SideLowerArm2
- removed link Torso
- added link Body0, mass 1; collision box size=0.8071791179959931 1.5211474410570394 0.25946855363821175; visual box size=0.8071791179959931 1.5211474410570394 0.25946855363821175
- added link Body1, mass 1; collision box size=2.1644163572090145 1.8520406648873078 0.9307348936795633; visual box size=2.1644163572090145 1.8520406648873078 0.9307348936795633
- added link Body2, mass 1; collision box size=2.256499663288963 1.1104902504383698 0.3181228526004959; visual box size=2.256499663288963 1.1104902504383698 0.3181228526004959
- added link Body3, mass 1; collision box size=0.11840914919928547 0.9773843912284466 0.0070553803409899585; visual box size=0.11840914919928547 0.9773843912284466 0.0070553803409899585
- added link Body4, mass 1; collision box size=0.35262133817112884 1.8413458808335286 0.49065921715489913; visual box size=0.35262133817112884 1.8413458808335286 0.49065921715489913
- added link Body5, mass 1; collision box size=2.153187243423364 0.2187053612232679 0.8292127454966207; visual box size=2.153187243423364 0.2187053612232679 0.8292127454966207
Joints:
- removed joint LeftLeg1_LeftLowerLeg1
- removed joint LeftLeg2_LeftLowerLeg2
- removed joint RightLeg1_RightLowerLeg1
- removed joint RightLeg2_RightLowerLeg2
- removed joint SideArm1_SideLowerArm1
- removed joint SideArm2_SideLowerArm2
- removed joint Torso_LeftLeg1
- removed joint Torso_LeftLeg2
- removed joint Torso_RightLeg1
- removed joint Torso_RightLeg2
- removed joint Torso_SideArm1
- removed joint Torso_SideArm2
- added joint Body0_Body1: type revolute, parent Body0, child Body1, origin xyz=1.5964104410020035 0.0 0.5 rpy=0 0 0, axis 0 1 0, limit lower=-3.14159 upper=3.14159 effort=0.0 velocity=0.0
- added joint Body1_Body2: type revolute, parent Body1, child Body2, origin xyz=-2.1644163572090145 0.0 0.0 rpy=0 0 0, axis 0 1 0, limit lower=-3.14159 upper=3.14159 effort=0.0 velocity=0.0
- added joint Body2_Body3: type revolute, parent Body2, child Body3, origin xyz=-2.256499663288963 0.0 0.0 rpy=0 0 0, axis 0 1 0, limit lower=-3.14159 upper=3.14159 effort=0.0 velocity=0.0
- added joint Body3_Body4: type revolute, parent Body3, child Body4, origin xyz=-0.11840914919928547 0.0 0.0 rpy=0 0 0, axis 0 1 0, limit lower=-3.14159 upper=3.14159 effort=0.0 velocity=0.0
- added joint Body4_Body5: type revolute, parent Body4, child Body5, origin xyz=-0.35262133817112884 0.0 0.0 rpy=0 0 0, axis 0 1 0, limit lower=-3.14159 upper=3.14159 effort=0.0 velocity=0.0

Commit message: made left side legs

File: body.urdf (robot description, URDF)
Before this commit: robot robot, 6 links, 5 joints
Links:
- added link Body6, mass 1; collision box size=0.2 0.2 0.4; visual box size=0.2 0.2 0.4
- added link Body7, mass 1; collision box size=0.2 0.5 0.2; visual box size=0.2 0.5 0.2
- added link Body8, mass 1; collision box size=0.2 0.2 0.4; visual box size=0.2 0.2 0.4
- link Body0: geometry collision box size=4 1 0.5; visual box size=4 1 0.5
- link Body1: geometry collision box size=0.2 0.5 0.2; visual box size=0.2 0.5 0.2
- link Body2: geometry collision box size=0.2 0.2 0.4; visual box size=0.2 0.2 0.4
- link Body3: geometry collision box size=0.2 0.5 0.2; visual box size=0.2 0.5 0.2
- link Body4: geometry collision box size=0.2 0.2 0.4; visual box size=0.2 0.2 0.4
- link Body5: geometry collision box size=0.2 0.5 0.2; visual box size=0.2 0.5 0.2
Joints:
- removed joint Body2_Body3
- removed joint Body4_Body5
- added joint Body0_Body3: type revolute, parent Body0, child Body3, origin xyz=-2.5 -0.5 0.45 rpy=0 0 0, axis 0 0 1, limit lower=-3.14159 upper=3.14159 effort=0.0 velocity=0.0
- added joint Body0_Body5: type revolute, parent Body0, child Body5, origin xyz=-1.5 -0.5 0.45 rpy=0 0 0, axis 0 0 1, limit lower=-3.14159 upper=3.14159 effort=0.0 velocity=0.0
- added joint Body0_Body7: type revolute, parent Body0, child Body7, origin xyz=-0.5 -0.5 0.45 rpy=0 0 0, axis 0 0 1, limit lower=-3.14159 upper=3.14159 effort=0.0 velocity=0.0
- added joint Body5_Body6: type revolute, parent Body5, child Body6, origin xyz=0 -0.5 0 rpy=0 0 0, axis 0 0 1, limit lower=-3.14159 upper=3.14159 effort=0.0 velocity=0.0
- added joint Body7_Body8: type revolute, parent Body7, child Body8, origin xyz=0 -0.5 0 rpy=0 0 0, axis 0 0 1, limit lower=-3.14159 upper=3.14159 effort=0.0 velocity=0.0
- joint Body0_Body1: axis 0 1 0 -> 0 0 1; origin xyz=1.5964104410020035 0.0 0.5 rpy=0 0 0 -> xyz=-3.5 -0.5 0.45 rpy=0 0 0
- joint Body1_Body2: axis 0 1 0 -> 0 0 1; origin xyz=-2.1644163572090145 0.0 0.0 rpy=0 0 0 -> xyz=0 -0.5 0 rpy=0 0 0
- joint Body3_Body4: axis 0 1 0 -> 0 0 1; origin xyz=-0.11840914919928547 0.0 0.0 rpy=0 0 0 -> xyz=0 -0.5 0 rpy=0 0 0

Commit message: just need to randomly pick sensor neurons

File: body.urdf (robot description, URDF)
Before this commit: robot robot, 9 links, 8 joints
Links:
- added link Body10, mass 1; collision box size=0.2 0.2 0.4; visual box size=0.2 0.2 0.4
- added link Body11, mass 1; collision box size=0.2 0.5 0.2; visual box size=0.2 0.5 0.2
- added link Body12, mass 1; collision box size=0.2 0.2 0.4; visual box size=0.2 0.2 0.4
- added link Body9, mass 1; collision box size=0.2 0.5 0.2; visual box size=0.2 0.5 0.2
- link Body0: geometry collision box size=3 1 0.5; visual box size=3 1 0.5
Joints:
- added joint Body0_Body11: type revolute, parent Body0, child Body11, origin xyz=-0.75 0.5 0.45 rpy=0 0 0, axis 0 0 1, limit lower=-3.14159 upper=3.14159 effort=0.0 velocity=0.0
- added joint Body0_Body9: type revolute, parent Body0, child Body9, origin xyz=-1.5 0.5 0.45 rpy=0 0 0, axis 0 0 1, limit lower=-3.14159 upper=3.14159 effort=0.0 velocity=0.0
- added joint Body11_Body12: type revolute, parent Body11, child Body12, origin xyz=0 0.5 0 rpy=0 0 0, axis 0 0 1, limit lower=-3.14159 upper=3.14159 effort=0.0 velocity=0.0
- added joint Body9_Body10: type revolute, parent Body9, child Body10, origin xyz=0 0.5 0 rpy=0 0 0, axis 0 0 1, limit lower=-3.14159 upper=3.14159 effort=0.0 velocity=0.0
- joint Body0_Body1: origin xyz=-3.5 -0.5 0.45 rpy=0 0 0 -> xyz=-2.25 -0.5 0.45 rpy=0 0 0
- joint Body0_Body3: origin xyz=-2.5 -0.5 0.45 rpy=0 0 0 -> xyz=-1.5 -0.5 0.45 rpy=0 0 0
- joint Body0_Body5: origin xyz=-1.5 -0.5 0.45 rpy=0 0 0 -> xyz=-0.75 -0.5 0.45 rpy=0 0 0
- joint Body0_Body7: origin xyz=-0.5 -0.5 0.45 rpy=0 0 0 -> xyz=-2.25 0.5 0.45 rpy=0 0 0
- joint Body7_Body8: origin xyz=0 -0.5 0 rpy=0 0 0 -> xyz=0 0.5 0 rpy=0 0 0

Commit message: expands in 2D so far

File: body.urdf (robot description, URDF)
Before this commit: robot robot, 6 links, 5 joints
Links:
- added link Body10, mass 1; collision box size=0.39159066358636757 0.717666905411628 0.1697063569241156; visual box size=0.39159066358636757 0.717666905411628 0.1697063569241156
- added link Body11, mass 1; collision box size=0.22742107160184 0.8973180085644421 0.010849993152315598; visual box size=0.22742107160184 0.8973180085644421 0.010849993152315598
- added link Body6, mass 1; collision box size=0.18943258466494073 0.4996282006102486 0.06651477491919293; visual box size=0.18943258466494073 0.4996282006102486 0.06651477491919293
- added link Body7, mass 1; collision box size=0.11783437991606557 0.8664852286139189 0.4078561760045503; visual box size=0.11783437991606557 0.8664852286139189 0.4078561760045503
- added link Body8, mass 1; collision box size=1.0625998174257472 0.23755969979852076 0.14343424052872022; visual box size=1.0625998174257472 0.23755969979852076 0.14343424052872022
- added link Body9, mass 1; collision box size=2.1755075489825106 1.2357736934377723 0.18109953160694803; visual box size=2.1755075489825106 1.2357736934377723 0.18109953160694803
- link Body0: geometry collision box size=2.861869787592354 0.16230550001222332 0.8097093014815109; visual box size=2.861869787592354 0.16230550001222332 0.8097093014815109
- link Body1: geometry collision box size=0.8532502223263996 0.6009979109019972 0.09566293598560116; visual box size=0.8532502223263996 0.6009979109019972 0.09566293598560116
- link Body2: geometry collision box size=1.5151298143122613 0.6731351598681057 0.4155380266732306; visual box size=1.5151298143122613 0.6731351598681057 0.4155380266732306
- link Body3: geometry collision box size=0.5096973771461515 0.16549812731283708 0.13630680666456074; visual box size=0.5096973771461515 0.16549812731283708 0.13630680666456074
- link Body4: geometry collision box size=0.2213659644292542 0.9934262768154403 0.2555649414283706; visual box size=0.2213659644292542 0.9934262768154403 0.2555649414283706
- link Body5: geometry collision box size=0.8944253380786347 0.906557355961616 0.6319532021364057; visual box size=0.8944253380786347 0.906557355961616 0.6319532021364057
Joints:
- added joint Body10_Body11: type revolute, parent Body10, child Body11, origin xyz=0.0 1.2357736934377723 0.0 rpy=0 0 0, axis 0 1 0, limit lower=-3.14159 upper=3.14159 effort=0.0 velocity=0.0
- added joint Body5_Body6: type revolute, parent Body5, child Body6, origin xyz=-0.44721266903931733 -0.453278677980808 0.0 rpy=0 0 0, axis 0 1 0, limit lower=-3.14159 upper=3.14159 effort=0.0 velocity=0.0
- added joint Body6_Body7: type revolute, parent Body6, child Body7, origin xyz=0.0 0.906557355961616 0.0 rpy=0 0 0, axis 0 1 0, limit lower=-3.14159 upper=3.14159 effort=0.0 velocity=0.0
- added joint Body7_Body8: type revolute, parent Body7, child Body8, origin xyz=-0.44721266903931733 -0.453278677980808 0.0 rpy=0 0 0, axis 0 1 0, limit lower=-3.14159 upper=3.14159 effort=0.0 velocity=0.0
- added joint Body8_Body9: type revolute, parent Body8, child Body9, origin xyz=-1.0625998174257472 0.0 0.0 rpy=0 0 0, axis 0 1 0, limit lower=-3.14159 upper=3.14159 effort=0.0 velocity=0.0
- added joint Body9_Body10: type revolute, parent Body9, child Body10, origin xyz=-1.0877537744912553 -0.6178868467188862 0.0 rpy=0 0 0, axis 0 1 0, limit lower=-3.14159 upper=3.14159 effort=0.0 velocity=0.0
- joint Body0_Body1: origin xyz=1.5964104410020035 0.0 0.5 rpy=0 0 0 -> xyz=0.569065106203823 0.0 0.5 rpy=0 0 0
- joint Body1_Body2: origin xyz=-2.1644163572090145 0.0 0.0 rpy=0 0 0 -> xyz=-0.8532502223263996 0.0 0.0 rpy=0 0 0
- joint Body2_Body3: origin xyz=-2.256499663288963 0.0 0.0 rpy=0 0 0 -> xyz=-0.7575649071561307 -0.33656757993405284 0.0 rpy=0 0 0
- joint Body3_Body4: origin xyz=-0.11840914919928547 0.0 0.0 rpy=0 0 0 -> xyz=0.0 0.6731351598681057 0.0 rpy=0 0 0
- joint Body4_Body5: origin xyz=-0.35262133817112884 0.0 0.0 rpy=0 0 0 -> xyz=-0.7575649071561307 -0.33656757993405284 0.0 rpy=0 0 0
