Commit message: produces legs

File: body.urdf (robot description, URDF)
Before this commit: robot robot, 12 links, 11 joints
Links:
- added link Body12, mass 1; collision box size=0.12966644772125094 1.831226518368709 0.3353641025668043; visual box size=0.12966644772125094 1.831226518368709 0.3353641025668043
- added link Body13, mass 1; collision box size=0.12966644772125094 0.9156132591843545 0.5; visual box size=0.12966644772125094 0.9156132591843545 0.5
- added link Body14, mass 1; collision box size=0.026729639242211358 0.7148011433388248 0.029807890880375363; visual box size=0.026729639242211358 0.7148011433388248 0.029807890880375363
- added link Body15, mass 1; collision box size=0.026729639242211358 0.3574005716694124 0.5; visual box size=0.026729639242211358 0.3574005716694124 0.5
- added link Body16, mass 1; collision box size=2.6046639709923776 0.567880848001838 0.8338234509017347; visual box size=2.6046639709923776 0.567880848001838 0.8338234509017347
- added link Body17, mass 1; collision box size=0.15268046395801604 0.4557462733112476 0.8251342268959918; visual box size=0.15268046395801604 0.4557462733112476 0.8251342268959918
- added link Body18, mass 1; collision box size=0.15268046395801604 0.2278731366556238 0.5; visual box size=0.15268046395801604 0.2278731366556238 0.5
- added link Body19, mass 1; collision box size=1.1450066653558264 0.9830319772341245 0.30499014319434475; visual box size=1.1450066653558264 0.9830319772341245 0.30499014319434475
- added link Body20, mass 1; collision box size=1.1450066653558264 0.49151598861706225 0.5; visual box size=1.1450066653558264 0.49151598861706225 0.5
- added link Body21, mass 1; collision box size=1.1336772184466286 0.043089211096427604 0.6043399187150553; visual box size=1.1336772184466286 0.043089211096427604 0.6043399187150553
- added link Body22, mass 1; collision box size=0.15212660837358213 0.059960669738541084 0.5946943453435014; visual box size=0.15212660837358213 0.059960669738541084 0.5946943453435014
- added link Body23, mass 1; collision box size=0.15212660837358213 0.029980334869270542 0.5; visual box size=0.15212660837358213 0.029980334869270542 0.5
- added link Body24, mass 1; collision box size=0.2697420647060007 1.6645638993482288 0.21669607748892494; visual box size=0.2697420647060007 1.6645638993482288 0.21669607748892494
- added link Body25, mass 1; collision box size=0.2697420647060007 0.8322819496741144 0.5; visual box size=0.2697420647060007 0.8322819496741144 0.5
- link Body0: geometry collision box size=1.7174171325425494 1.8074058492705711 0.6554370983193305; visual box size=1.7174171325425494 1.8074058492705711 0.6554370983193305
- link Body1: geometry collision box size=2.524893744836147 1.0277036109938238 0.8534568903573734; visual box size=2.524893744836147 1.0277036109938238 0.8534568903573734
- link Body10: geometry collision box size=0.6692248971421628 0.6358130745615919 0.5; visual box size=0.6692248971421628 0.6358130745615919 0.5
- link Body11: geometry collision box size=0.6402937864354429 0.13280849908005443 0.39055173399402443; visual box size=0.6402937864354429 0.13280849908005443 0.39055173399402443
- link Body2: geometry collision box size=0.6906735418387882 1.4229958235200175 0.548323162845989; visual box size=0.6906735418387882 1.4229958235200175 0.548323162845989
- link Body3: geometry collision box size=0.6906735418387882 0.7114979117600088 0.5; visual box size=0.6906735418387882 0.7114979117600088 0.5
- link Body4: geometry collision box size=0.5993256404398629 0.9265322278307166 0.6602251018801432; visual box size=0.5993256404398629 0.9265322278307166 0.6602251018801432
- link Body5: geometry collision box size=0.5993256404398629 0.4632661139153583 0.5; visual box size=0.5993256404398629 0.4632661139153583 0.5
- link Body6: geometry collision box size=1.564522872465922 1.2903780506464622 0.04201168758982954; visual box size=1.564522872465922 1.2903780506464622 0.04201168758982954
- link Body7: geometry collision box size=0.14413370264367875 0.40684733311587973 0.0348181483489102; visual box size=0.14413370264367875 0.40684733311587973 0.0348181483489102
- link Body8: geometry collision box size=0.14413370264367875 0.20342366655793986 0.5; visual box size=0.14413370264367875 0.20342366655793986 0.5
- link Body9: geometry collision box size=0.6692248971421628 1.2716261491231837 0.023969191809200985; visual box size=0.6692248971421628 1.2716261491231837 0.023969191809200985
Joints:
- added joint Body11_Body12: type revolute, parent Body11, child Body12, origin xyz=-0.32014689321772144 -0.06640424954002722 0.0 rpy=0 0 0, axis 0 1 0, limit lower=-3.14159 upper=3.14159 effort=0.0 velocity=0.0
- added joint Body12_Body13: type revolute, parent Body12, child Body13, origin xyz=0.0 -1.831226518368709 0.0 rpy=0 0 0, axis 0 0 1, limit lower=-3.14159 upper=3.14159 effort=0.0 velocity=0.0
- added joint Body13_Body14: type revolute, parent Body13, child Body14, origin xyz=0.0 1.9640350174487635 0.0 rpy=0 0 0, axis 0 0 1, limit lower=-3.14159 upper=3.14159 effort=0.0 velocity=0.0
- added joint Body14_Body15: type revolute, parent Body14, child Body15, origin xyz=0.0 0.7148011433388248 0.0 rpy=0 0 0, axis 0 0 1, limit lower=-3.14159 upper=3.14159 effort=0.0 velocity=0.0
- added joint Body15_Body16: type revolute, parent Body15, child Body16, origin xyz=-0.32014689321772144 -0.781205392878852 0.0 rpy=0 0 0, axis 0 1 0, limit lower=-3.14159 upper=3.14159 effort=0.0 velocity=0.0
- added joint Body16_Body17: type revolute, parent Body16, child Body17, origin xyz=-1.3023319854961888 -0.283940424000919 0.0 rpy=0 0 0, axis 0 1 0, limit lower=-3.14159 upper=3.14159 effort=0.0 velocity=0.0
- added joint Body17_Body18: type revolute, parent Body17, child Body18, origin xyz=0.0 -0.4557462733112476 0.0 rpy=0 0 0, axis 0 0 1, limit lower=-3.14159 upper=3.14159 effort=0.0 velocity=0.0
- added joint Body18_Body19: type revolute, parent Body18, child Body19, origin xyz=0.0 1.0236271213130856 0.0 rpy=0 0 0, axis 0 0 1, limit lower=-3.14159 upper=3.14159 effort=0.0 velocity=0.0
- added joint Body19_Body20: type revolute, parent Body19, child Body20, origin xyz=0.0 0.9830319772341245 0.0 rpy=0 0 0, axis 0 0 1, limit lower=-3.14159 upper=3.14159 effort=0.0 velocity=0.0
- added joint Body20_Body21: type revolute, parent Body20, child Body21, origin xyz=-1.3023319854961888 -1.2669724012350434 0.0 rpy=0 0 0, axis 0 1 0, limit lower=-3.14159 upper=3.14159 effort=0.0 velocity=0.0
- added joint Body21_Body22: type revolute, parent Body21, child Body22, origin xyz=-0.5668386092233143 -0.021544605548213802 0.0 rpy=0 0 0, axis 0 1 0, limit lower=-3.14159 upper=3.14159 effort=0.0 velocity=0.0
- added joint Body22_Body23: type revolute, parent Body22, child Body23, origin xyz=0.0 -0.059960669738541084 0.0 rpy=0 0 0, axis 0 0 1, limit lower=-3.14159 upper=3.14159 effort=0.0 velocity=0.0
- added joint Body23_Body24: type revolute, parent Body23, child Body24, origin xyz=0.0 0.10304988083496869 0.0 rpy=0 0 0, axis 0 0 1, limit lower=-3.14159 upper=3.14159 effort=0.0 velocity=0.0
- added joint Body24_Body25: type revolute, parent Body24, child Body25, origin xyz=0.0 1.6645638993482288 0.0 rpy=0 0 0, axis 0 0 1, limit lower=-3.14159 upper=3.14159 effort=0.0 velocity=0.0
- joint Body0_Body1: origin xyz=0.569065106203823 0.0 0.5 rpy=0 0 0 -> xyz=1.1412914337287252 0.0 0.5 rpy=0 0 0
- joint Body10_Body11: origin xyz=0.0 1.2357736934377723 0.0 rpy=0 0 0 -> xyz=-0.782261436232961 -1.9168151744464148 0.0 rpy=0 0 0
- joint Body1_Body2: origin xyz=-0.8532502223263996 0.0 0.0 rpy=0 0 0 -> xyz=-1.2624468724180735 -0.5138518054969119 0.0 rpy=0 0 0
- joint Body2_Body3: axis 0 1 0 -> 0 0 1; origin xyz=-0.7575649071561307 -0.33656757993405284 0.0 rpy=0 0 0 -> xyz=0.0 -1.4229958235200175 0.0 rpy=0 0 0
- joint Body3_Body4: axis 0 1 0 -> 0 0 1; origin xyz=0.0 0.6731351598681057 0.0 rpy=0 0 0 -> xyz=0.0 2.450699434513841 0.0 rpy=0 0 0
- joint Body4_Body5: axis 0 1 0 -> 0 0 1; origin xyz=-0.7575649071561307 -0.33656757993405284 0.0 rpy=0 0 0 -> xyz=0.0 0.9265322278307166 0.0 rpy=0 0 0
- joint Body5_Body6: origin xyz=-0.44721266903931733 -0.453278677980808 0.0 rpy=0 0 0 -> xyz=-1.2624468724180735 -1.4403840333276285 0.0 rpy=0 0 0
- joint Body6_Body7: origin xyz=0.0 0.906557355961616 0.0 rpy=0 0 0 -> xyz=-0.782261436232961 -0.6451890253232311 0.0 rpy=0 0 0
- joint Body7_Body8: axis 0 1 0 -> 0 0 1; origin xyz=-0.44721266903931733 -0.453278677980808 0.0 rpy=0 0 0 -> xyz=0.0 -0.40684733311587973 0.0 rpy=0 0 0
- joint Body8_Body9: axis 0 1 0 -> 0 0 1; origin xyz=-1.0625998174257472 0.0 0.0 rpy=0 0 0 -> xyz=0.0 1.6972253837623419 0.0 rpy=0 0 0
- joint Body9_Body10: axis 0 1 0 -> 0 0 1; origin xyz=-1.0877537744912553 -0.6178868467188862 0.0 rpy=0 0 0 -> xyz=0.0 1.2716261491231837 0.0 rpy=0 0 0

Commit message: finished left leg

File: body.urdf (robot description, URDF)
Before this commit: robot robot, 26 links, 25 joints
Links:
- removed link Body10
- removed link Body11
- removed link Body12
- removed link Body13
- removed link Body14
- removed link Body15
- removed link Body16
- removed link Body17
- removed link Body18
- removed link Body19
- removed link Body20
- removed link Body21
- removed link Body22
- removed link Body23
- removed link Body24
- removed link Body25
- removed link Body5
- removed link Body6
- removed link Body7
- removed link Body8
- removed link Body9
- link Body0: geometry collision box size=0.9242580823102231 1.68720313983972 0.7559997484969235; visual box size=0.9242580823102231 1.68720313983972 0.7559997484969235
- link Body1: geometry collision box size=1 1.5813371171167776 0.3449359502636926; visual box size=1 1.5813371171167776 0.3449359502636926
- link Body2: geometry collision box size=0.7211964874160018 0.06132610815598317 0.1724679751318463; visual box size=0.7211964874160018 0.06132610815598317 0.1724679751318463
- link Body3: geometry collision box size=1 1 0.5259190923866426; visual box size=1 1 0.5259190923866426
- link Body4: geometry collision box size=0.7244272337570189 0.7325359170521109 0.2629595461933213; visual box size=0.7244272337570189 0.7325359170521109 0.2629595461933213
Joints:
- removed joint Body10_Body11
- removed joint Body11_Body12
- removed joint Body12_Body13
- removed joint Body13_Body14
- removed joint Body14_Body15
- removed joint Body15_Body16
- removed joint Body16_Body17
- removed joint Body17_Body18
- removed joint Body18_Body19
- removed joint Body19_Body20
- removed joint Body20_Body21
- removed joint Body21_Body22
- removed joint Body22_Body23
- removed joint Body23_Body24
- removed joint Body24_Body25
- removed joint Body2_Body3
- removed joint Body4_Body5
- removed joint Body5_Body6
- removed joint Body6_Body7
- removed joint Body7_Body8
- removed joint Body8_Body9
- removed joint Body9_Body10
- added joint Body1_Body3: type revolute, parent Body1, child Body3, origin xyz=-1 0 0 rpy=0 0 0, axis 0 1 0, limit lower=-3.14159 upper=3.14159 effort=0.0 velocity=0.0
- joint Body0_Body1: origin xyz=1.1412914337287252 0.0 0.5 rpy=0 0 0 -> xyz=1.5378709588448884 0 0.5 rpy=0 0 0
- joint Body1_Body2: origin xyz=-1.2624468724180735 -0.5138518054969119 0.0 rpy=0 0 0 -> xyz=-0.5 -0.7906685585583888 0 rpy=0 0 0
- joint Body3_Body4: axis 0 0 1 -> 0 1 0; origin xyz=0.0 2.450699434513841 0.0 rpy=0 0 0 -> xyz=-0.5 -0.5 0 rpy=0 0 0

Commit message: made lizard!

File: body.urdf (robot description, URDF)
Before this commit: robot robot, 5 links, 4 joints
Links:
- added link Body5, mass 1; collision box size=0.42482457242187044 0.6933666941963116 0.3855180055553603; visual box size=0.42482457242187044 0.6933666941963116 0.3855180055553603
- link Body0: geometry collision box size=0.3889374345460195 1.6024912105956906 0.45921078994107023; visual box size=0.3889374345460195 1.6024912105956906 0.45921078994107023
- link Body1: geometry collision box size=1.7781346518976615 1.0024753725149955 0.3330588102039824; visual box size=1.7781346518976615 1.0024753725149955 0.3330588102039824
- link Body2: geometry collision box size=0.8588153064230836 0.13075422733270106 0.1665294051019912; visual box size=0.8588153064230836 0.13075422733270106 0.1665294051019912
- link Body3: geometry collision box size=1 1.5169145135529576 0.7710360111107206; visual box size=1 1.5169145135529576 0.7710360111107206
- link Body4: geometry collision box size=0.9811117158864482 0.3729811852243625 0.3855180055553603; visual box size=0.9811117158864482 0.3729811852243625 0.3855180055553603
Joints:
- added joint Body3_Body5: type revolute, parent Body3, child Body5, origin xyz=-0.5 0.7584572567764788 0 rpy=0 0 0, axis 0 0 1, limit lower=-3.14159 upper=3.14159 effort=0.0 velocity=0.0
- joint Body0_Body1: origin xyz=1.5378709588448884 0 0.5 rpy=0 0 0 -> xyz=1.8055312827269903 0 0.5 rpy=0 0 0
- joint Body1_Body2: axis 0 1 0 -> 0 0 1; origin xyz=-0.5 -0.7906685585583888 0 rpy=0 0 0 -> xyz=-0.8890673259488308 0.5012376862574978 0 rpy=0 0 0
- joint Body1_Body3: origin xyz=-1 0 0 rpy=0 0 0 -> xyz=-1.7781346518976615 0 0 rpy=0 0 0
- joint Body3_Body4: axis 0 1 0 -> 0 0 1; origin xyz=-0.5 -0.5 0 rpy=0 0 0 -> xyz=-0.5 -0.7584572567764788 0 rpy=0 0 0

Commit message: finished refactoring

File: body.urdf (robot description, URDF)
Before this commit: robot robot, 6 links, 5 joints
Links:
- added link Body6, mass 1; collision box size=0.3248153831687025 0.3945906369021278 0.75; visual box size=0.3248153831687025 0.3945906369021278 0.75
- link Body0: geometry collision box size=1.7903888614579089 1.1345498168741506 0.7065307055180984; visual box size=1.7903888614579089 1.1345498168741506 0.7065307055180984
- link Body1: geometry collision box size=1 1 0.2743686521315132; visual box size=1 1 0.2743686521315132
- link Body2: geometry collision box size=0.07775367537651678 0.9832746461946191 0.1371843260657566; visual box size=0.07775367537651678 0.9832746461946191 0.1371843260657566
- link Body3: geometry collision box size=0.07775367537651678 0.49163732309730956 0.75; visual box size=0.07775367537651678 0.49163732309730956 0.75
- link Body4: geometry collision box size=1.4750387491381294 1.0138078382937505 0.2549654516803236; visual box size=1.4750387491381294 1.0138078382937505 0.2549654516803236
- link Body5: geometry collision box size=0.3248153831687025 0.7891812738042556 0.1274827258401618; visual box size=0.3248153831687025 0.7891812738042556 0.1274827258401618
Joints:
- removed joint Body1_Body3
- removed joint Body3_Body4
- removed joint Body3_Body5
- added joint Body1_Body4: type revolute, parent Body1, child Body4, origin xyz=-1 0 0 rpy=0 0 0, axis 0 1 0, limit lower=-3.14159 upper=3.14159 effort=0.0 velocity=0.0
- added joint Body2_Body3: type revolute, parent Body2, child Body3, origin xyz=0 0.9832746461946191 0 rpy=0 0 0, axis 0 0 1, limit lower=-3.14159 upper=3.14159 effort=0.0 velocity=0.0
- added joint Body4_Body5: type revolute, parent Body4, child Body5, origin xyz=-0.7375193745690647 -0.5069039191468753 0 rpy=0 0 0, axis 0 0 1, limit lower=-3.14159 upper=3.14159 effort=0.0 velocity=0.0
- added joint Body5_Body6: type revolute, parent Body5, child Body6, origin xyz=0 -0.7891812738042556 0 rpy=0 0 0, axis 0 0 1, limit lower=-3.14159 upper=3.14159 effort=0.0 velocity=0.0
- joint Body0_Body1: origin xyz=1.8055312827269903 0 0.5 rpy=0 0 0 -> xyz=1.1048055692710457 0 1.5 rpy=0 0 0
- joint Body1_Body2: origin xyz=-0.8890673259488308 0.5012376862574978 0 rpy=0 0 0 -> xyz=-0.5 0.5 0 rpy=0 0 0

Commit message: Finished assignment 8

File: body.urdf (robot description, URDF)
Before this commit: robot robot, 7 links, 6 joints
Links:
- added link Body7, mass 1; collision box size=0.8630455842896205 0.2812176312813339 0.06606042882961227; visual box size=0.8630455842896205 0.2812176312813339 0.06606042882961227
- added link Body8, mass 1; collision box size=0.8630455842896205 0.14060881564066696 0.75; visual box size=0.8630455842896205 0.14060881564066696 0.75
- link Body0: geometry collision box size=1.0278166829829836 0.7974601037175526 0.04794882306983772; visual box size=1.0278166829829836 0.7974601037175526 0.04794882306983772
- link Body1: geometry collision box size=1 1.2350852220030366 0.7690586001196474; visual box size=1 1.2350852220030366 0.7690586001196474
- link Body2: geometry collision box size=0.8807911124963281 0.5569556404157302 0.3845293000598237; visual box size=0.8807911124963281 0.5569556404157302 0.3845293000598237
- link Body3: geometry collision box size=0.8807911124963281 0.2784778202078651 0.75; visual box size=0.8807911124963281 0.2784778202078651 0.75
- link Body4: geometry collision box size=1.5893531301831376 1 0.13212085765922454; visual box size=1.5893531301831376 1 0.13212085765922454
- link Body5: geometry collision box size=0.6055969075017298 0.71766514009941 0.06606042882961227; visual box size=0.6055969075017298 0.71766514009941 0.06606042882961227
- link Body6: geometry collision box size=0.6055969075017298 0.358832570049705 0.75; visual box size=0.6055969075017298 0.358832570049705 0.75
Joints:
- added joint Body4_Body7: type revolute, parent Body4, child Body7, origin xyz=-0.7946765650915688 0.5 0 rpy=0 0 0, axis 0 0 1, limit lower=-3.14159 upper=3.14159 effort=0.0 velocity=0.0
- added joint Body7_Body8: type revolute, parent Body7, child Body8, origin xyz=0 0.2812176312813339 0 rpy=0 0 0, axis 0 0 1, limit lower=-3.14159 upper=3.14159 effort=0.0 velocity=0.0
- joint Body0_Body1: origin xyz=1.1048055692710457 0 1.5 rpy=0 0 0 -> xyz=1.4860916585085082 0 1.5 rpy=0 0 0
- joint Body1_Body2: origin xyz=-0.5 0.5 0 rpy=0 0 0 -> xyz=-0.5 -0.6175426110015183 0 rpy=0 0 0
- joint Body2_Body3: origin xyz=0 0.9832746461946191 0 rpy=0 0 0 -> xyz=0 -0.5569556404157302 0 rpy=0 0 0
- joint Body4_Body5: origin xyz=-0.7375193745690647 -0.5069039191468753 0 rpy=0 0 0 -> xyz=-0.7946765650915688 -0.5 0 rpy=0 0 0
- joint Body5_Body6: origin xyz=0 -0.7891812738042556 0 rpy=0 0 0 -> xyz=0 -0.71766514009941 0 rpy=0 0 0

Commit message: assignment 7

File: body.urdf (robot description, URDF)
Before this commit: robot robot, 26 links, 25 joints
Links:
- removed link Body16
- removed link Body17
- removed link Body18
- removed link Body19
- removed link Body20
- removed link Body21
- removed link Body22
- removed link Body23
- removed link Body24
- removed link Body25
- link Body0: geometry collision box size=0.5768442370087475 0.2341030456654396 0.3114277621222691; visual box size=0.5768442370087475 0.2341030456654396 0.3114277621222691
- link Body1: geometry collision box size=2.4165623673418017 0.5882980702318752 0.443183993097494; visual box size=2.4165623673418017 0.5882980702318752 0.443183993097494
- link Body10: geometry collision box size=1.0899427556885668 0.6459116683127886 0.5; visual box size=1.0899427556885668 0.6459116683127886 0.5
- link Body11: geometry collision box size=2.3333173372073914 0.9943426695400583 0.5144846694451446; visual box size=2.3333173372073914 0.9943426695400583 0.5144846694451446
- link Body12: geometry collision box size=0.9210809389695849 1.1126258466914645 0.20283383790344775; visual box size=0.9210809389695849 1.1126258466914645 0.20283383790344775
- link Body13: geometry collision box size=0.9210809389695849 0.5563129233457322 0.5; visual box size=0.9210809389695849 0.5563129233457322 0.5
- link Body14: geometry collision box size=0.5128233002150917 1.121772893349807 0.27970323376972117; visual box size=0.5128233002150917 1.121772893349807 0.27970323376972117
- link Body15: geometry collision box size=0.5128233002150917 0.5608864466749035 0.5; visual box size=0.5128233002150917 0.5608864466749035 0.5
- link Body2: geometry collision box size=1.0037635906342752 0.7891187897467553 0.21528863989796376; visual box size=1.0037635906342752 0.7891187897467553 0.21528863989796376
- link Body3: geometry collision box size=1.0037635906342752 0.39455939487337766 0.5; visual box size=1.0037635906342752 0.39455939487337766 0.5
- link Body4: geometry collision box size=0.09994915012065184 1.4078837325674114 0.08546226530251347; visual box size=0.09994915012065184 1.4078837325674114 0.08546226530251347
- link Body5: geometry collision box size=0.09994915012065184 0.7039418662837057 0.5; visual box size=0.09994915012065184 0.7039418662837057 0.5
- link Body6: geometry collision box size=2.6167452016771486 0.9346169810515088 0.22742040810752284; visual box size=2.6167452016771486 0.9346169810515088 0.22742040810752284
- link Body7: geometry collision box size=0.8236416471054655 0.24577950858508912 0.078648085873308; visual box size=0.8236416471054655 0.24577950858508912 0.078648085873308
- link Body8: geometry collision box size=0.8236416471054655 0.12288975429254456 0.5; visual box size=0.8236416471054655 0.12288975429254456 0.5
- link Body9: geometry collision box size=1.0899427556885668 1.2918233366255771 0.15553117261683602; visual box size=1.0899427556885668 1.2918233366255771 0.15553117261683602
Joints:
- removed joint Body15_Body16
- removed joint Body16_Body17
- removed joint Body17_Body18
- removed joint Body18_Body19
- removed joint Body19_Body20
- removed joint Body20_Body21
- removed joint Body21_Body22
- removed joint Body22_Body23
- removed joint Body23_Body24
- removed joint Body24_Body25
- joint Body0_Body1: origin xyz=1.1412914337287252 0.0 0.5 rpy=0 0 0 -> xyz=1.7115778814956262 0.0 0.5 rpy=0 0 0
- joint Body10_Body11: origin xyz=-0.782261436232961 -1.9168151744464148 0.0 rpy=0 0 0 -> xyz=-1.3083726008385743 -1.7591318271513314 0.0 rpy=0 0 0
- joint Body11_Body12: origin xyz=-0.32014689321772144 -0.06640424954002722 0.0 rpy=0 0 0 -> xyz=-1.1666586686036957 -0.49717133477002917 0.0 rpy=0 0 0
- joint Body12_Body13: origin xyz=0.0 -1.831226518368709 0.0 rpy=0 0 0 -> xyz=0.0 -1.1126258466914645 0.0 rpy=0 0 0
- joint Body13_Body14: origin xyz=0.0 1.9640350174487635 0.0 rpy=0 0 0 -> xyz=0.0 2.1069685162315226 0.0 rpy=0 0 0
- joint Body14_Body15: origin xyz=0.0 0.7148011433388248 0.0 rpy=0 0 0 -> xyz=0.0 1.121772893349807 0.0 rpy=0 0 0
- joint Body1_Body2: origin xyz=-1.2624468724180735 -0.5138518054969119 0.0 rpy=0 0 0 -> xyz=-1.2082811836709009 -0.2941490351159376 0.0 rpy=0 0 0
- joint Body2_Body3: origin xyz=0.0 -1.4229958235200175 0.0 rpy=0 0 0 -> xyz=0.0 -0.7891187897467553 0.0 rpy=0 0 0
- joint Body3_Body4: origin xyz=0.0 2.450699434513841 0.0 rpy=0 0 0 -> xyz=0.0 1.3774168599786305 0.0 rpy=0 0 0
- joint Body4_Body5: origin xyz=0.0 0.9265322278307166 0.0 rpy=0 0 0 -> xyz=0.0 1.4078837325674114 0.0 rpy=0 0 0
- joint Body5_Body6: origin xyz=-1.2624468724180735 -1.4403840333276285 0.0 rpy=0 0 0 -> xyz=-1.2082811836709009 -1.7020327676833489 0.0 rpy=0 0 0
- joint Body6_Body7: origin xyz=-0.782261436232961 -0.6451890253232311 0.0 rpy=0 0 0 -> xyz=-1.3083726008385743 -0.4673084905257544 0.0 rpy=0 0 0
- joint Body7_Body8: origin xyz=0.0 -0.40684733311587973 0.0 rpy=0 0 0 -> xyz=0.0 -0.24577950858508912 0.0 rpy=0 0 0
- joint Body8_Body9: origin xyz=0.0 1.6972253837623419 0.0 rpy=0 0 0 -> xyz=0.0 1.180396489636598 0.0 rpy=0 0 0
- joint Body9_Body10: origin xyz=0.0 1.2716261491231837 0.0 rpy=0 0 0 -> xyz=0.0 1.2918233366255771 0.0 rpy=0 0 0
