Commit message: got 3 parts

File: body.urdf (robot description, URDF)
Before this commit: robot robot, 16 links, 15 joints
Links:
- removed link Body0
- removed link Body1
- removed link Body10
- removed link Body11
- removed link Body12
- removed link Body13
- removed link Body14
- removed link Body15
- removed link Body2
- removed link Body3
- removed link Body4
- removed link Body5
- removed link Body6
- removed link Body7
- removed link Body8
- removed link Body9
- added link spine0, mass 1; collision box size=0.5414571417848075 0.2804988775982946 0.6140713137525462; visual box size=0.5414571417848075 0.2804988775982946 0.6140713137525462
Joints:
- removed joint Body0_Body1
- removed joint Body10_Body11
- removed joint Body11_Body12
- removed joint Body12_Body13
- removed joint Body13_Body14
- removed joint Body14_Body15
- removed joint Body1_Body2
- removed joint Body2_Body3
- removed joint Body3_Body4
- removed joint Body4_Body5
- removed joint Body5_Body6
- removed joint Body6_Body7
- removed joint Body7_Body8
- removed joint Body8_Body9
- removed joint Body9_Body10
- added joint spine0_arm0: type revolute, parent spine0, child _arm0, origin xyz=-0.27072857089240376 -0.1402494387991473 0.0 rpy=0 0 0, axis 0 1 0, limit lower=-3.14159 upper=3.14159 effort=0.0 velocity=0.0

Commit message: testing order

File: body.urdf (robot description, URDF)
Before this commit: robot robot, 3 links, 2 joints
Links:
- added link Arm, mass 1; collision box size=1 1 1; visual box size=1 1 1
Joints:
- added joint BackLeg_Arm: type rotate, parent BackLeg, child Arm, origin xyz=-0.5 -0.5 -0.5 rpy=0 0 0, axis 0 1 0, limit lower=-3.14159 upper=3.14159 effort=0.0 velocity=0.0
